File: integration_elec/integration_elec_master/MCU.kicad_sch (KiCad schematic)
At the start: 20 parts, among them SW1 SW_Push, U2 STM32F446RETx, Y1 Crystal_16MHz

Commit message: Added switch in design + Footprint + symbol
Connections:
- net VALVE1_ON: now reaches U2.39 (PC8)
- net VALVE2_ON: now reaches U2.40 (PC9)
Other:
- note added: "PULL UP PC8 PC9"
