File: integration_elec/integration_elec_master/TFT_SCREEN AND JOYSTICK.kicad_sch (KiCad schematic)
At the start: 2 parts, among them U5 COM-28379, U6 COM-09032

Commit message: Added switch in design + Footprint + symbol
Parts:
- added S1, S2: RB141C1100, SWITCH:SW_RB141C1100, symbol RB141C1100:RB141C1100
Connections:
- net GND: now also S1.1, S2.1
- new net VALVE1_ON: S1.2
- new net VALVE2_ON: S2.2
