File: integration_elec/integration_elec_master/integration_elec_master.kicad_sch (KiCad schematic)
At the start: 0 parts

Commit message: KAH - Fini schematic attente de review + correction BUS
Other:
- sheet DEBUG_USB ports: added {DEBUG}, {USB}; removed none
- sheet MCU ports: added RF{XBEE}, {DEBUG}, {JOYSTICK}, {TFT_SCREEN}, {USB}; removed none
- sheet TFT_SCREEN AND JOYSTICK ports: added {JOYSTICK}, {TFT_SCREEN}; removed none
- sheet XBEE ports: added RF{XBEE}; removed none
Changed lines of the file:
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@@
 	(generator_version "9.0")
 	(paper "A4")
+	(bus
+		(pts
+			(xy 106.68 106.68) (xy 106.68 121.92)
+		)
+		(stroke
+			(width 0)
+			(type default)
+		)
+	)
+	(bus
+		(pts
+			(xy 101.6 106.68) (xy 101.6 121.92)
+		)
+		(stroke
+			(width 0)
+			(type default)
+		)
+	)
+	(bus
+		(pts
+			(xy 101.6 68.58) (xy 101.6 80.01)
+		)
+		(stroke
+			(width 0)
+			(type default)
+		)
+	)
+	(bus
+		(pts
+			(xy 124.46 88.9) (xy 139.7 88.9)
+		)
+		(stroke
+			(width 0)
+			(type default)
+		)
+	)
+	(bus
+		(pts
+			(xy 124.46 99.06) (xy 139.7 99.06)
+		)
+		(stroke
+			(width 0)
+			(type default)
+		)
+	)
 	(sheet
 		(at 63.5 121.92)
@@
 				)
 				(justify left top)
+			)
+		)
+		(pin "{JOYSTICK}" bidirectional
+			(at 101.6 121.92 90)
+			(effects
+				(font
+					(size 1.27 1.27)
+				)
+				(justify right)
+			)
+		)
+		(pin "{TFT_SCREEN}" bidirectional
+			(at 106.68 121.92 90)
+			(effects
+				(font
+					(size 1.27 1.27)
+				)
+				(justify right)
 			)
 		)
@@
 			)
 		)
+		(pin "RF{XBEE}" bidirectional
+			(at 101.6 80.01 90)
+			(effects
+				(font
+					(size 1.27 1.27)
+				)
+				(justify right)
+			)
+		)
+		(pin "{DEBUG}" bidirectional
+			(at 124.46 99.06 0)
+			(effects
+				(font
+					(size 1.27 1.27)
+				)
+				(justify right)
+			)
+		)
+		(pin "{JOYSTICK}" bidirectional
+			(at 101.6 106.68 270)
+			(effects
+				(font
+					(size 1.27 1.27)
+				)
+				(justify left)
+			)
+		)
+		(pin "{TFT_SCREEN}" bidirectional
+			(at 106.68 106.68 270)
+			(effects
+				(font
+					(size 1.27 1.27)
+				)
+				(justify left)
+			)
+		)
+		(pin "{USB}" bidirectional
+			(at 124.46 88.9 0)
+			(effects
+				(font
+					(size 1.27 1.27)
+				)
+				(justify right)
+			)
+		)
 		(instances
 			(project "integration_elec_master"
@@
 			)
 		)
+		(pin "RF{XBEE}" bidirectional
+			(at 101.6 68.58 270)
+			(effects
+				(font
+					(size 1.27 1.27)
+				)
+				(justify left)
+			)
+		)
 		(instances
 			(project "integration_elec_master"
@@
 	)
 	(sheet
-		(at 151.765 78.74)
-		(size 60.96 28.575)
+		(at 139.7 41.91)
+		(size 60.325 28.575)
 		(exclude_from_sim no)
 		(in_bom yes)
@@
 		)
 		(property "Sheetname" "REGULATOR"
-			(at 151.765 78.0284 0)
+			(at 139.7 41.1984 0)
 			(effects
 				(font
@@
 		)
 		(property "Sheetfile" "REGULATOR.kicad_sch"
-			(at 151.765 107.8996 0)
+			(at 139.7 71.0696 0)
 			(effects
 				(font
@@
 	)
 	(sheet
-		(at 151.13 41.275)
-		(size 60.325 25.4)
+		(at 139.7 80.01)
+		(size 60.325 26.67)
 		(exclude_from_sim no)
 		(in_bom yes)
@@
 		)
 		(property "Sheetname" "DEBUG_USB"
-			(at 151.13 40.5634 0)
+			(at 139.7 79.2984 0)
 			(effects
 				(font
@@
 		)
 		(property "Sheetfile" "DEBUG_USB.kicad_sch"
-			(at 151.13 67.2596 0)
-			(effects
-				(font
-					(size 1.27 1.27)
-				)
-				(justify left top)
-			)
-		)
+			(at 139.7 107.2646 0)
+			(effects
+				(font
+					(size 1.27 1.27)
+				)
+				(justify left top)
+			)
+		)
+		(pin "{DEBUG}" bidirectional
+			(at 139.7 99.06 180)
+			(effects
+				(font
+					(size 1.27 1.27)
+				)
+				(justify left)
+			)
+		)
+		(pin "{USB}" output
+			(at 139.7 88.9 180)
+			(effects
+				(font
+					(size 1.27 1.27)
+				)
+				(justify left)
+			)
+		)

Commit message: EM - Review finale (final i guess)
Parts:
- added H1, H2, H3, H4: MountingHole, MountingHole:MountingHole_3.2mm_M3, symbol Mechanical:MountingHole
