File: integration_elec/integration_elec_slave/XBEE.kicad_sch (KiCad schematic)
At the start: 12 parts, among them Q1 Q_NMOS_GSD, U2 XBEE_PRO_900HP

Commit message: EM - fuck it we merge et on cree deux branches
Parts:
- renumbered C13 to C1, C14 to C2, C17 to C3, C15 to C4, C16 to C5, R58 to R1, R4 to R2, R34 to R3, R5 to R4, U2 to U1
Changed lines of the file:
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@@
 		(on_board yes)
 		(dnp no)
-		(property "Reference" "U2"
+		(property "Reference" "U1"
 			(at 154.305 80.1878 0)
 			(effects
@@
 			(project "integration_elec_slave"
 				(path "/f8f45849-17b1-4cdb-b0ac-47b1208e44f3/b0a0cc4c-fc88-458b-9c77-f065f39e4cf1"
-					(reference "U2")
+					(reference "U1")
 					(unit 1)
 				)
@@
 		(on_board yes)
 		(dnp no)
-		(property "Reference" "#PWR011"
+		(property "Reference" "#PWR04"
 			(at 125.73 78.74 0)
 			(effects
@@
 			(project "integration_elec_slave"
 				(path "/f8f45849-17b1-4cdb-b0ac-47b1208e44f3/b0a0cc4c-fc88-458b-9c77-f065f39e4cf1"
-					(reference "#PWR011")
+					(reference "#PWR04")
 					(unit 1)
 				)
@@
 		(on_board yes)
 		(dnp no)
-		(property "Reference" "#PWR017"
+		(property "Reference" "#PWR05"
 			(at 125.73 121.92 0)
 			(effects
@@
 			(project "integration_elec_slave"
 				(path "/f8f45849-17b1-4cdb-b0ac-47b1208e44f3/b0a0cc4c-fc88-458b-9c77-f065f39e4cf1"
-					(reference "#PWR017")
+					(reference "#PWR05")
 					(unit 1)
 				)
@@
 		(on_board yes)
 		(dnp no)
-		(property "Reference" "#PWR015"
+		(property "Reference" "#PWR01"
 			(at 80.01 101.6 0)
 			(effects
@@
 			(project "integration_elec_slave"
 				(path "/f8f45849-17b1-4cdb-b0ac-47b1208e44f3/b0a0cc4c-fc88-458b-9c77-f065f39e4cf1"
-					(reference "#PWR015")
+					(reference "#PWR01")
 					(unit 1)
 				)
@@
 		(on_board yes)
 		(dnp no)
-		(property "Reference" "C17"
+		(property "Reference" "C3"
 			(at 103.0732 111.6584 0)
 			(effects
@@
 			(project "integration_elec_slave"
 				(path "/f8f45849-17b1-4cdb-b0ac-47b1208e44f3/b0a0cc4c-fc88-458b-9c77-f065f39e4cf1"
-					(reference "C17")
+					(reference "C3")
 					(unit 1)
 				)
@@
 		(on_board yes)
 		(dnp no)
-		(property "Reference" "#PWR016"
+		(property "Reference" "#PWR03"
 			(at 105.41 121.92 0)
 			(effects
@@
 			(project "integration_elec_slave"
 				(path "/f8f45849-17b1-4cdb-b0ac-47b1208e44f3/b0a0cc4c-fc88-458b-9c77-f065f39e4cf1"
-					(reference "#PWR016")
+					(reference "#PWR03")
 					(unit 1)
 				)
@@
 		(on_board yes)
 		(dnp no)
-		(property "Reference" "#PWR012"
+		(property "Reference" "#PWR06"
 			(at 179.07 81.28 0)
 			(effects
@@
 			(project "integration_elec_slave"
 				(path "/f8f45849-17b1-4cdb-b0ac-47b1208e44f3/b0a0cc4c-fc88-458b-9c77-f065f39e4cf1"
-					(reference "#PWR012")
+					(reference "#PWR06")
 					(unit 1)
 				)
@@
 		(on_board yes)
 		(dnp no)
-		(property "Reference" "R4"
+		(property "Reference" "R2"
 			(at 191.77 88.9 90)
 			(effects
@@
 			(project "integration_elec_slave"
 				(path "/f8f45849-17b1-4cdb-b0ac-47b1208e44f3/b0a0cc4c-fc88-458b-9c77-f065f39e4cf1"
-					(reference "R4")
+					(reference "R2")
 					(unit 1)
 				)
@@
 		(on_board yes)
 		(dnp no)
-		(property "Reference" "#PWR018"
+		(property "Reference" "#PWR09"
 			(at 234.95 134.62 0)
 			(effects
@@
 			(project "integration_elec_slave"
 				(path "/f8f45849-17b1-4cdb-b0ac-47b1208e44f3/b0a0cc4c-fc88-458b-9c77-f065f39e4cf1"
-					(reference "#PWR018")
+					(reference "#PWR09")
 					(unit 1)
 				)
@@
 		(on_board yes)
 		(dnp no)
-		(property "Reference" "R5"
+		(property "Reference" "R4"
 			(at 239.395 102.87 0)
 			(effects
@@
 			(project "integration_elec_slave"
 				(path "/f8f45849-17b1-4cdb-b0ac-47b1208e44f3/b0a0cc4c-fc88-458b-9c77-f065f39e4cf1"
-					(reference "R5")
+					(reference "R4")
 					(unit 1)
 				)
@@
 		(on_board yes)
 		(dnp no)
-		(property "Reference" "#PWR014"
+		(property "Reference" "#PWR08"
 			(at 234.95 93.98 0)
 			(effects
@@
 			(project "integration_elec_slave"
 				(path "/f8f45849-17b1-4cdb-b0ac-47b1208e44f3/b0a0cc4c-fc88-458b-9c77-f065f39e4cf1"
-					(reference "#PWR014")
+					(reference "#PWR08")
 					(unit 1)
 				)
@@
 		(on_board yes)
 		(dnp no)
-		(property "Reference" "R34"
+		(property "Reference" "R3"
 			(at 223.52 125.73 90)
 			(effects
@@
 			(project "integration_elec_slave"
 				(path "/f8f45849-17b1-4cdb-b0ac-47b1208e44f3/b0a0cc4c-fc88-458b-9c77-f065f39e4cf1"
-					(reference "R34")
+					(reference "R3")
 					(unit 1)
 				)
@@
 		(on_board yes)
 		(dnp no)
-		(property "Reference" "#PWR0101"
+		(property "Reference" "#PWR07"
 			(at 222.25 134.62 0)
 			(effects
@@
 			(project "integration_elec_slave"
 				(path "/f8f45849-17b1-4cdb-b0ac-47b1208e44f3/b0a0cc4c-fc88-458b-9c77-f065f39e4cf1"
-					(reference "#PWR0101")
+					(reference "#PWR07")
 					(unit 1)
 				)
@@
 		(on_board yes)
 		(dnp no)
-		(property "Reference" "R58"
+		(property "Reference" "R1"
 			(at 182.245 80.645 0)
 			(effects
@@
 			(project "integration_elec_slave"
 				(path "/f8f45849-17b1-4cdb-b0ac-47b1208e44f3/b0a0cc4c-fc88-458b-9c77-f065f39e4cf1"
-					(reference "R58")
+					(reference "R1")
 					(unit 1)
 				)
@@
 		(on_board yes)
 		(dnp no)
-		(property "Reference" "C16"
+		(property "Reference" "C5"
 			(at 120.65 83.82 0)
 			(effects
@@
 			(project "integration_elec_slave"
 				(path "/f8f45849-17b1-4cdb-b0ac-47b1208e44f3/b0a0cc4c-fc88-458b-9c77-f065f39e4cf1"
-					(reference "C16")
+					(reference "C5")
 					(unit 1)
 				)
@@
 		(on_board yes)
 		(dnp no)
-		(property "Reference" "#PWR013"
+		(property "Reference" "#PWR02"
 			(at 87.63 93.98 0)
 			(effects
@@
 			(project "integration_elec_slave"
 				(path "/f8f45849-17b1-4cdb-b0ac-47b1208e44f3/b0a0cc4c-fc88-458b-9c77-f065f39e4cf1"
-					(reference "#PWR013")
+					(reference "#PWR02")
 					(unit 1)
 				)
@@
 		(on_board yes)
 		(dnp no)
-		(property "Reference" "C15"
+		(property "Reference" "C4"
 			(at 113.2332 83.7184 0)
 			(effects
@@
 			(project "integration_elec_slave"
 				(path "/f8f45849-17b1-4cdb-b0ac-47b1208e44f3/b0a0cc4c-fc88-458b-9c77-f065f39e4cf1"
-					(reference "C15")
+					(reference "C4")
 					(unit 1)
 				)
@@
 		(dnp no)
 		(fields_autoplaced yes)
-		(property "Reference" "C13"
+		(property "Reference" "C1"
 			(at 90.17 81.2736 0)
 			(effects
@@
 			(project "integration_elec_slave"
 				(path "/f8f45849-17b1-4cdb-b0ac-47b1208e44f3/b0a0cc4c-fc88-458b-9c77-f065f39e4cf1"
-					(reference "C13")
+					(reference "C1")
 					(unit 1)
 				)
@@
 		(on_board yes)
 		(dnp no)
-		(property "Reference" "C14"
+		(property "Reference" "C2"
 			(at 100.5332 83.7184 0)
 			(effects
@@
 			(project "integration_elec_slave"
 				(path "/f8f45849-17b1-4cdb-b0ac-47b1208e44f3/b0a0cc4c-fc88-458b-9c77-f065f39e4cf1"
-					(reference "C14")
-					(unit 1)
-				)
+					(reference "C2")
+					(unit 1)
+				)

Commit message: EM - Fini schématique attente de review
Parts:
- removed R3: 10k, Resistor_SMD:R_0805_2012Metric_Pad1.20x1.40mm_HandSolder, symbol Device:R_US
- added R34: 10k, Resistor_SMD:R_0805_2012Metric_Pad1.20x1.40mm_HandSolder, symbol Device:R_US
Connections:
- net GND: now also R2.2
- net RF.XBEE_LED: now also R2.1
- net RF.XBEE_RQ: now also R34.1; no longer R2.1
- net at R1.2, U1.9 (nDTR): now also R34.2; no longer R2.2
