File: integration_elec/integration_elec_slave/integration_elec_slave.kicad_pcb (KiCad board)
At the start: 4 copper layers, 0 parts

Commit message: EM - Fini schématique attente de review
Parts:
- added C1: 10uF, Capacitor_SMD:C_0805_2012Metric_Pad1.18x1.45mm_HandSolder, F.Cu at (204.3, 49.5)
- added C10: 4.7uF, Capacitor_SMD:C_0805_2012Metric_Pad1.18x1.45mm_HandSolder, F.Cu at (155.8, 114.2)
- added C11: 0.10uF, Capacitor_SMD:C_0805_2012Metric_Pad1.18x1.45mm_HandSolder, F.Cu at (155.8, 117.2)
- added C12: 0.10uF, Capacitor_SMD:C_0805_2012Metric_Pad1.18x1.45mm_HandSolder, F.Cu at (155.8, 120.2)
- added C13: 0.10uF, Capacitor_SMD:C_0805_2012Metric_Pad1.18x1.45mm_HandSolder, F.Cu at (155.8, 123.3)
- added C14: 0.10uF, Capacitor_SMD:C_0805_2012Metric_Pad1.18x1.45mm_HandSolder, F.Cu at (160.6, 114.2)
- added C15: 0.10uF, Capacitor_SMD:C_0805_2012Metric_Pad1.18x1.45mm_HandSolder, F.Cu at (160.6, 117.2)
- added C16: 0.10uF, Capacitor_SMD:C_0805_2012Metric_Pad1.18x1.45mm_HandSolder, F.Cu at (160.6, 120.2)
- added C17: 0.10uF, Capacitor_SMD:C_0805_2012Metric_Pad1.18x1.45mm_HandSolder, F.Cu at (160.6, 123.3)
- added C18: 0.10uF, Capacitor_SMD:C_0805_2012Metric_Pad1.18x1.45mm_HandSolder, F.Cu at (223.0, 86.6)
- added C19: 0.10uF, Capacitor_SMD:C_0805_2012Metric_Pad1.18x1.45mm_HandSolder, F.Cu at (223.0, 89.6)
- added C2: 1uF, Capacitor_SMD:C_0805_2012Metric_Pad1.18x1.45mm_HandSolder, F.Cu at (204.3, 52.5)
- added C20: 10uF, Capacitor_SMD:C_0805_2012Metric_Pad1.18x1.45mm_HandSolder, F.Cu at (146.2, 78.4)
- added C21: 10uF, Capacitor_SMD:C_0805_2012Metric_Pad1.18x1.45mm_HandSolder, F.Cu at (146.2, 81.5)
- added C22: 10uF, Capacitor_SMD:C_0805_2012Metric_Pad1.18x1.45mm_HandSolder, F.Cu at (146.2, 84.5)
- added C23: 0.10uF, Capacitor_SMD:C_0805_2012Metric_Pad1.18x1.45mm_HandSolder, F.Cu at (146.2, 87.5)
- added C24: 6.8nF, Capacitor_SMD:C_0805_2012Metric_Pad1.18x1.45mm_HandSolder, F.Cu at (146.2, 90.5)
- added C25: 120pF, Capacitor_SMD:C_0805_2012Metric_Pad1.18x1.45mm_HandSolder, F.Cu at (151.0, 78.4)
- added C26: 0.10uF, Capacitor_SMD:C_0805_2012Metric_Pad1.18x1.45mm_HandSolder, F.Cu at (151.0, 81.5)
- added C27: 100 uF, Capacitor_SMD:C_1206_3216Metric, F.Cu at (161.1, 64.4)
- added C28: 100 uF, Capacitor_SMD:C_1206_3216Metric, F.Cu at (161.1, 67.8)
- added C29: 100 uF, Capacitor_SMD:C_1206_3216Metric, F.Cu at (161.1, 71.1)
- added C3: 10nF, Capacitor_SMD:C_0805_2012Metric_Pad1.18x1.45mm_HandSolder, F.Cu at (204.3, 55.5)
- added C30: 100 uF, Capacitor_SMD:C_1206_3216Metric, F.Cu at (161.1, 74.5)
- added C31: 100 uF, Capacitor_SMD:C_1206_3216Metric, F.Cu at (161.1, 77.8)
- added C32: 10uF, Capacitor_SMD:C_0805_2012Metric_Pad1.18x1.45mm_HandSolder, F.Cu at (151.0, 84.5)
- added C33: 10uF, Capacitor_SMD:C_0805_2012Metric_Pad1.18x1.45mm_HandSolder, F.Cu at (151.0, 87.5)
- added C34: 10uF, Capacitor_SMD:C_0805_2012Metric_Pad1.18x1.45mm_HandSolder, F.Cu at (151.0, 90.5)
- added C35: 0.10uF, Capacitor_SMD:C_0805_2012Metric_Pad1.18x1.45mm_HandSolder, F.Cu at (155.8, 78.4)
- added C36: 6.8nF, Capacitor_SMD:C_0805_2012Metric_Pad1.18x1.45mm_HandSolder, F.Cu at (155.8, 81.5)
- added C37: 120pF, Capacitor_SMD:C_0805_2012Metric_Pad1.18x1.45mm_HandSolder, F.Cu at (155.8, 84.5)
- added C38: 0.10uF, Capacitor_SMD:C_0805_2012Metric_Pad1.18x1.45mm_HandSolder, F.Cu at (155.8, 87.5)
- added C39: 100 uF, Capacitor_SMD:C_1206_3216Metric, F.Cu at (161.1, 81.2)
- added C4: 47pF, Capacitor_SMD:C_0805_2012Metric_Pad1.18x1.45mm_HandSolder, F.Cu at (204.3, 58.6)
- added C40: 100 uF, Capacitor_SMD:C_1206_3216Metric, F.Cu at (161.1, 84.5)
- added C41: 100 uF, Capacitor_SMD:C_1206_3216Metric, F.Cu at (161.1, 87.9)
- added C42: 100 uF, Capacitor_SMD:C_1206_3216Metric, F.Cu at (161.1, 91.2)
- added C43: 100 uF, Capacitor_SMD:C_1206_3216Metric, F.Cu at (161.1, 94.6)
- added C5: 10pF, Capacitor_SMD:C_0805_2012Metric_Pad1.18x1.45mm_HandSolder, F.Cu at (204.3, 61.6)
- added C6: 10pF, Capacitor_SMD:C_0805_2012Metric_Pad1.18x1.45mm_HandSolder, F.Cu at (150.9, 114.2)
- added C7: 0.10uF, Capacitor_SMD:C_0805_2012Metric_Pad1.18x1.45mm_HandSolder, F.Cu at (150.9, 117.2)
- added C8: 10pF, Capacitor_SMD:C_0805_2012Metric_Pad1.18x1.45mm_HandSolder, F.Cu at (150.9, 120.2)
- added C9: 0.10uF, Capacitor_SMD:C_0805_2012Metric_Pad1.18x1.45mm_HandSolder, F.Cu at (150.9, 123.3)
- added D1: BLUE LED, LED_SMD:LED_0805_2012Metric_Pad1.15x1.40mm_HandSolder, F.Cu at (204.3, 80.8)
- added D2: BLUE LED, LED_SMD:LED_0805_2012Metric_Pad1.15x1.40mm_HandSolder, F.Cu at (171.0, 77.6)
- added J1: CONN_02X05, Esteban11:CONN_CNC_10_pins, F.Cu at (210.6, 89.1)
- added J2: USB_C_Receptacle_USB2.0_16P, Connector_USB:USB_C_Receptacle_GCT_USB4105-xx-A_16P_TopMnt_Horizontal, F.Cu at (210.5, 97.4)
- added J3: Conn_01x03_Pin, Connector_Molex:Molex_Micro-Fit_3.0_43650-0315_1x03_P3.00mm_Vertical, F.Cu at (213.1, 67.2)
- added J4: Conn_01x04_Pin, Connector_Molex:Molex_Micro-Fit_3.0_43650-0415_1x04_P3.00mm_Vertical, F.Cu at (213.1, 51.5)
- added J5: Conn_01x04_Pin, Connector_Molex:Molex_Micro-Fit_3.0_43650-0415_1x04_P3.00mm_Vertical, F.Cu at (213.1, 59.3)
- added L1: FerritBead 600 OHM, Inductor_SMD:L_0805_2012Metric_Pad1.15x1.40mm_HandSolder, F.Cu at (146.2, 99.7)
- added L2: 15 uH, Inductors:IND_BOURNS_SRR1280, F.Cu at (151.0, 55.3)
- added L3: 15 uH, Inductors:IND_BOURNS_SRR1280, F.Cu at (151.0, 69.7)
- added Q1: Q_NMOS_GSD, Package_TO_SOT_SMD:SOT-23, F.Cu at (204.3, 77.1)
- added Q2: Q_NMOS_GSD, Package_TO_SOT_SMD:SOT-23, F.Cu at (177.8, 109.3)
- added Q3: Q_NMOS_GSD, Package_TO_SOT_SMD:SOT-23, F.Cu at (177.8, 113.8)
- added R1: NC, Resistor_SMD:R_0805_2012Metric_Pad1.20x1.40mm_HandSolder, F.Cu at (204.3, 64.5)
- added R10: 22, Resistor_SMD:R_0805_2012Metric_Pad1.20x1.40mm_HandSolder, F.Cu at (218.7, 96.5)
- added R11: 5.1K, Resistor_SMD:R_0603_1608Metric_Pad0.98x0.95mm_HandSolder, F.Cu at (223.2, 93.4)
- added R12: 5.1K, Resistor_SMD:R_0603_1608Metric_Pad0.98x0.95mm_HandSolder, F.Cu at (223.2, 95.9)
- added R13: 1M, Resistor_SMD:R_0805_2012Metric_Pad1.20x1.40mm_HandSolder, F.Cu at (218.7, 99.5)
- added R14: NC, Resistor_SMD:R_0805_2012Metric_Pad1.20x1.40mm_HandSolder, F.Cu at (160.6, 49.5)
- added R15: NC, Resistor_SMD:R_0805_2012Metric_Pad1.20x1.40mm_HandSolder, F.Cu at (160.6, 52.4)
- added R16: 220k, Resistor_SMD:R_0805_2012Metric_Pad1.20x1.40mm_HandSolder, F.Cu at (160.6, 55.4)
- added R17: 10k, Resistor_SMD:R_0805_2012Metric_Pad1.20x1.40mm_HandSolder, F.Cu at (160.6, 58.3)
- added R18: 100k, Resistor_SMD:R_0805_2012Metric_Pad1.20x1.40mm_HandSolder, F.Cu at (160.6, 61.3)
- added R19: 31k6, Resistor_SMD:R_0805_2012Metric_Pad1.20x1.40mm_HandSolder, F.Cu at (165.4, 49.5)
- added R2: 10k, Resistor_SMD:R_0805_2012Metric_Pad1.20x1.40mm_HandSolder, F.Cu at (204.3, 67.5)
- added R20: 330, Resistor_SMD:R_0805_2012Metric_Pad1.20x1.40mm_HandSolder, F.Cu at (165.4, 52.4)
- added R21: 2.2k, Resistor_SMD:R_0805_2012Metric_Pad1.20x1.40mm_HandSolder, F.Cu at (211.2, 75.0)
- added R22: 20k, Resistor_SMD:R_0805_2012Metric_Pad1.20x1.40mm_HandSolder, F.Cu at (211.2, 77.9)
- added R23: 10k, Resistor_SMD:R_0805_2012Metric_Pad1.20x1.40mm_HandSolder, F.Cu at (211.2, 80.9)
- added R24: 10k, Resistor_SMD:R_0805_2012Metric_Pad1.20x1.40mm_HandSolder, F.Cu at (146.2, 114.5)
- added R25: 10k, Resistor_SMD:R_0805_2012Metric_Pad1.20x1.40mm_HandSolder, F.Cu at (146.2, 117.4)
- added R26: NC, Resistor_SMD:R_0805_2012Metric_Pad1.20x1.40mm_HandSolder, F.Cu at (165.4, 55.4)
- added R27: NC, Resistor_SMD:R_0805_2012Metric_Pad1.20x1.40mm_HandSolder, F.Cu at (165.4, 58.3)
- added R28: 220k, Resistor_SMD:R_0805_2012Metric_Pad1.20x1.40mm_HandSolder, F.Cu at (165.4, 61.3)
- added R29: 10k, Resistor_SMD:R_0805_2012Metric_Pad1.20x1.40mm_HandSolder, F.Cu at (170.1, 49.5)
- added R3: 10k, Resistor_SMD:R_0805_2012Metric_Pad1.20x1.40mm_HandSolder, F.Cu at (182.6, 108.6)
- added R30: 100k, Resistor_SMD:R_0805_2012Metric_Pad1.20x1.40mm_HandSolder, F.Cu at (170.1, 52.4)
- added R31: 19.1k, Resistor_SMD:R_0805_2012Metric_Pad1.20x1.40mm_HandSolder, F.Cu at (170.1, 55.4)
- added R32: 10k, Resistor_SMD:R_0805_2012Metric_Pad1.20x1.40mm_HandSolder, F.Cu at (182.6, 111.5)
- added R34: 10k, Resistor_SMD:R_0805_2012Metric_Pad1.20x1.40mm_HandSolder, F.Cu at (204.3, 73.4)
- added R4: 330, Resistor_SMD:R_0805_2012Metric_Pad1.20x1.40mm_HandSolder, F.Cu at (204.3, 70.4)
- added R5: 120, Resistor_SMD:R_0805_2012Metric_Pad1.20x1.40mm_HandSolder, F.Cu at (146.2, 102.7)
- added R6: 10k, Resistor_SMD:R_0805_2012Metric_Pad1.20x1.40mm_HandSolder, F.Cu at (146.2, 105.6)
- added R7: 10k, Resistor_SMD:R_0805_2012Metric_Pad1.20x1.40mm_HandSolder, F.Cu at (146.2, 108.6)
- added R8: 10k, Resistor_SMD:R_0805_2012Metric_Pad1.20x1.40mm_HandSolder, F.Cu at (146.2, 111.5)
- added R9: 22, Resistor_SMD:R_0805_2012Metric_Pad1.20x1.40mm_HandSolder, F.Cu at (218.7, 93.6)
- added SW1: SW_Push, Button_Switch_SMD:SW_SPST_TL3342, F.Cu at (167.8, 101.8)
- added TP1: GND, TestPoint:TestPoint_Plated_Hole_D2.0mm, F.Cu at (166.2, 78.4)
- added TP2: TestPoint, TestPoint:TestPoint_Plated_Hole_D2.0mm, F.Cu at (166.2, 83.1)
- added TP3: TestPoint, TestPoint:TestPoint_Plated_Hole_D2.0mm, F.Cu at (166.2, 87.7)
- added U1: XBEE_PRO_900HP, specific:XBEE_900HP, F.Cu at (177.5, 57.5)
- added U2: STM32F446RETx, Package_QFP:LQFP-64_10x10mm_P0.5mm, F.Cu at (155.8, 105.5)
- added U3: USBLC6-2SC6, Package_TO_SOT_SMD:SOT-23-6, F.Cu at (218.9, 103.4)
- added U4: TPS54335ADDAR, Package_SO:TI_SO-PowerPAD-8_ThermalVias, F.Cu at (168.2, 66.2)
- added U5: ADS1015IDGS, Package_SO:TSSOP-10_3x3mm_P0.5mm, F.Cu at (217.0, 75.8)
- added U6: J104D2C12VDC.20S, RELAY:RELAY8_J104D2C12VDC.20S_CRS, F.Cu at (179.4, 87.2)
- added U7: J104D2C12VDC.20S, RELAY:RELAY8_J104D2C12VDC.20S_CRS, F.Cu at (193.0, 87.2)
- added U8: TPS54335ADDAR, Package_SO:TI_SO-PowerPAD-8_ThermalVias, F.Cu at (168.2, 72.8)
- added Y1: Crystal_16MHz, ab2_xtal:CSM-3X, F.Cu at (168.0, 115.8)
