File: integration_elec/integration_elec_slave/GESTION_ALIM.kicad_sch (KiCad schematic)
At the start: 6 parts, among them Q2 Q_NMOS_GSD, Q3 Q_NMOS_GSD, U6 J104D2C12VDC.20S, U7 J104D2C12VDC.20S

Commit message: EM - Attente de review, complété avec les 3D
Parts:
- U6, U7: footprint RELAY8_J104D2C12VDC.20S_CRS -> RELAYS:RELAY8_J104D2C12VDC.20S_CRS
Changed lines of the file:
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@@
 			)
 		)
-		(property "Footprint" "RELAY8_J104D2C12VDC.20S_CRS"
+		(property "Footprint" "RELAYS:RELAY8_J104D2C12VDC.20S_CRS"
 			(at 116.84 57.15 0)
 			(effects
@@
 			)
 		)
-		(property "Footprint" "RELAY8_J104D2C12VDC.20S_CRS"
+		(property "Footprint" "RELAYS:RELAY8_J104D2C12VDC.20S_CRS"
 			(at 116.84 90.17 0)
 			(effects
